Commit message: Capstone modifications final fix

File: open_manipulator_description/gazebo/omy_f3m.gazebo.xacro (robot description, xacro)
@@ -6,9 +6,9 @@
       <type>transmission_interface/SimpleTransmission</type>
       <joint name="${joint}">
-        <hardwareInterface>PositionJointInterface</hardwareInterface>
+        <hardwareInterface>EffortJointInterface</hardwareInterface>
       </joint>
       <actuator name="${actuator}">
         <mechanicalReduction>1</mechanicalReduction>
-        <hardwareInterface>PositionJointInterface</hardwareInterface>
+        <hardwareInterface>EffortJointInterface</hardwareInterface>
       </actuator>
     </transmission>
@@ -24,4 +24,5 @@
     </gazebo>
   </xacro:macro>
+  <gazebo><self_collide>false</self_collide></gazebo>
   <xacro:Link reference="${prefix}link0"/>
   <xacro:Link reference="${prefix}link1"/>

File: open_manipulator_description/ros2_control/omy_f3m_current.ros2_control.xacro (robot description, xacro)
@@ -1,35 +1,9 @@
 <?xml version="1.0"?>
 <robot xmlns:xacro="http://www.ros.org/wiki/xacro">
-  <xacro:macro name="omy_f3m_system" params="name prefix port_name:=^|/dev/ttyAMA2 use_sim:=^|false use_mock_hardware:=^|false mock_sensor_commands:=^|false">
-    <ros2_control name="${name}" type="system" is_async="true">
-      <xacro:if value="$(arg use_sim)">
-        <hardware>
-          <plugin>gz_ros2_control/GazeboSimSystem</plugin>
-        </hardware>
-      </xacro:if>
-      <xacro:unless value="$(arg use_sim)">
-        <hardware>
-          <xacro:if value="${use_mock_hardware}">
-            <plugin>mock_components/GenericSystem</plugin>
-            <param name="mock_sensor_commands">${mock_sensor_commands}</param>
-            <param name="state_following_offset">0.0</param>
-          </xacro:if>
-          <xacro:unless value="${use_mock_hardware}">
-            <plugin>dynamixel_hardware_interface/DynamixelHardware</plugin>
-            <param name="port_name">${port_name}</param>
-            <param name="baud_rate">6250000</param>
-            <param name="error_timeout_ms">500</param>
-            <param name="dynamixel_model_folder">/param/dxl_model</param>
-            <param name="number_of_joints">6</param>
-            <param name="number_of_transmissions">6</param>
-            <param name="disable_torque_at_init">true</param>
-            <param name="dynamixel_state_pub_msg_name">dynamixel_hardware_interface/dxl_state</param>
-            <param name="get_dynamixel_data_srv_name">dynamixel_hardware_interface/get_dxl_data</param>
-            <param name="set_dynamixel_data_srv_name">dynamixel_hardware_interface/set_dxl_data</param>
-            <param name="reboot_dxl_srv_name">dynamixel_hardware_interface/reboot_dxl</param>
-            <param name="set_dxl_torque_srv_name">dynamixel_hardware_interface/set_dxl_torque</param>
-          </xacro:unless>
-        </hardware>
-      </xacro:unless>
+  <xacro:macro name="omy_f3m_system" params="name prefix port_name:=^|/dev/ttyUSB0 use_sim:=^|false use_mock_hardware:=^|false mock_sensor_commands:=^|false">
+    <ros2_control name="${name}" type="system">
+      <hardware>
+        <plugin>gz_ros2_control/GazeboSimSystem</plugin>
+      </hardware>
       <joint name="${prefix}joint1">
         <command_interface name="effort"/>
@@ -68,149 +42,10 @@
         <state_interface name="effort"/>
       </joint>
-      <gpio name="omy_hat">
-        <param name="type">controller</param>
-        <param name="ID">200</param>
-        <param name="Power Enable">1</param>
-        <param name="Voltage Control Enable">1</param>
-        <param name="R LED">200</param>
-        <param name="G LED">200</param>
-        <param name="B LED">120</param>
-        <param name="Baud Rate (Bus)">8</param>
-        <param name="DXL Baud Rate">8</param>
-        <param name="Status">0</param>
-      </gpio>
-      <gpio name="dxl1">
-        <param name="type">dxl</param>
-        <param name="ID">1</param>
-        <command_interface name="Goal Current"/>
-        <state_interface name="Present Position"/>
-        <state_interface name="Present Velocity"/>
-        <state_interface name="Present Current"/>
-        <param name="Torque Enable">1</param>
-        <param name="Drive Mode">4</param>
-        <param name="Velocity Limit">3591</param>
-        <param name="Acceleration Limit">8050</param>
-        <param name="Profile Velocity">3591</param>
-        <param name="Profile Acceleration">8050</param>
-        <param name="Homing Offset">0</param>
-        <param name="Return Delay Time">0</param>
-        <param name="Position P Gain">1583185</param>
-        <param name="Velocity P Gain">41387</param>
-        <param name="Velocity I Gain">1565630</param>
-        <param name="Operating Mode">0</param>
-        <param name="Profile Acceleration Time">20</param>
-        <param name="Profile Time">40</param>
-        <param name="Bus Watchdog">1</param>
-      </gpio>
-      <gpio name="dxl2">
-        <param name="type">dxl</param>
-        <param name="ID">2</param>
-        <command_interface name="Goal Current"/>
-        <state_interface name="Present Position"/>
-        <state_interface name="Present Velocity"/>
-        <state_interface name="Present Current"/>
-        <param name="Torque Enable">1</param>
-        <param name="Drive Mode">5</param>
-        <param name="Velocity Limit">3591</param>
-        <param name="Acceleration Limit">8050</param>
-        <param name="Profile Velocity">3591</param>
-        <param name="Profile Acceleration">8050</param>
-        <param name="Return Delay Time">0</param>
-        <param name="Position P Gain">1583185</param>
-        <param name="Velocity P Gain">41387</param>
-        <param name="Velocity I Gain">1565630</param>
-        <param name="Operating Mode">0</param>
-        <param name="Profile Acceleration Time">20</param>
-        <param name="Profile Time">40</param>
-        <param name="Bus Watchdog">1</param>
-      </gpio>
-      <gpio name="dxl3">
-        <param name="type">dxl</param>
-        <param name="ID">3</param>
-        <command_interface name="Goal Current"/>
-        <state_interface name="Present Position"/>
-        <state_interface name="Present Velocity"/>
-        <state_interface name="Present Current"/>
-        <param name="Torque Enable">1</param>
-        <param name="Drive Mode">4</param>
-        <param name="Velocity Limit">6486</param>
-        <param name="Acceleration Limit">8050</param>
-        <param name="Profile Velocity">6486</param>
-        <param name="Profile Acceleration">8050</param>
-        <param name="Return Delay Time">0</param>
-        <param name="Position P Gain">1583185</param>
-        <param name="Velocity P Gain">18184</param>
-        <param name="Velocity I Gain">1585331</param>
-        <param name="Operating Mode">0</param>
-        <param name="Profile Acceleration Time">20</param>
-        <param name="Profile Time">40</param>
-        <param name="Bus Watchdog">1</param>
-      </gpio>
-      <gpio name="dxl4">
-        <param name="type">dxl</param>
-        <param name="ID">4</param>
-        <command_interface name="Goal Current"/>
-        <state_interface name="Present Position"/>
-        <state_interface name="Present Velocity"/>
-        <state_interface name="Present Current"/>
-        <param name="Torque Enable">1</param>
-        <param name="Drive Mode">5</param>
-        <param name="Velocity Limit">6486</param>
-        <param name="Acceleration Limit">8050</param>
-        <param name="Profile Velocity">6486</param>
-        <param name="Profile Acceleration">8050</param>
-        <param name="Return Delay Time">0</param>
-        <param name="Position P Gain">1583185</param>
-        <param name="Velocity P Gain">18184</param>
-        <param name="Velocity I Gain">1585331</param>
-        <param name="Operating Mode">0</param>
-        <param name="Profile Acceleration Time">20</param>
-        <param name="Profile Time">40</param>
-        <param name="Bus Watchdog">1</param>
-      </gpio>
-      <gpio name="dxl5">
-        <param name="type">dxl</param>
-        <param name="ID">5</param>
-        <command_interface name="Goal Current"/>
-        <state_interface name="Present Position"/>
-        <state_interface name="Present Velocity"/>
-        <state_interface name="Present Current"/>
-        <param name="Torque Enable">1</param>
-        <param name="Drive Mode">4</param>
-        <param name="Velocity Limit">6486</param>
-        <param name="Acceleration Limit">8050</param>
-        <param name="Profile Velocity">6486</param>
-        <param name="Profile Acceleration">8050</param>
-        <param name="Return Delay Time">0</param>
-        <param name="Position P Gain">1583185</param>
-        <param name="Velocity P Gain">18184</param>
-        <param name="Velocity I Gain">1585331</param>
-        <param name="Operating Mode">0</param>
-        <param name="Profile Acceleration Time">20</param>
-        <param name="Profile Time">40</param>
-        <param name="Bus Watchdog">1</param>
-      </gpio>
-      <gpio name="dxl6">
-        <param name="type">dxl</param>
-        <param name="ID">6</param>
-        <command_interface name="Goal Current"/>
-        <state_interface name="Present Position"/>
-        <state_interface name="Present Velocity"/>
-        <state_interface name="Present Current"/>
-        <param name="Torque Enable">1</param>
-        <param name="Drive Mode">5</param>
-        <param name="Velocity Limit">6486</param>
-        <param name="Acceleration Limit">8050</param>
-        <param name="Profile Velocity">6486</param>
-        <param name="Profile Acceleration">8050</param>
-        <param name="Return Delay Time">0</param>
-        <param name="Position P Gain">1583185</param>
-        <param name="Velocity P Gain">18184</param>
-        <param name="Velocity I Gain">1585331</param>
-        <param name="Operating Mode">0</param>
-        <param name="Profile Acceleration Time">20</param>
-        <param name="Profile Time">40</param>
-        <param name="Bus Watchdog">1</param>
-      </gpio>
+      <joint name="${prefix}rh_r1_joint">
+        <command_interface name="effort"/>
+        <state_interface name="position"/>
+        <state_interface name="velocity"/>
+        <state_interface name="effort"/>
+      </joint>
     </ros2_control>
   </xacro:macro>

File: open_manipulator_description/ros2_control/omy_l100_current.ros2_control.xacro (robot description, xacro)
@@ -1,6 +1,6 @@
 <?xml version="1.0"?>
 <robot xmlns:xacro="http://www.ros.org/wiki/xacro">
-  <xacro:macro name="omy_l100_system" params="name prefix port_name:=^|/dev/ttyUSB0 use_sim:=^|false use_mock_hardware:=^|false mock_sensor_commands:=^|false">
-    <ros2_control name="${name}" type="system">
+  <xacro:macro name="omy_f3m_system" params="name prefix port_name:=^|/dev/ttyAMA2 use_sim:=^|false use_mock_hardware:=^|false mock_sensor_commands:=^|false">
+    <ros2_control name="${name}" type="system" is_async="true">
       <xacro:if value="$(arg use_sim)">
         <hardware>
@@ -18,9 +18,9 @@
             <plugin>dynamixel_hardware_interface/DynamixelHardware</plugin>
             <param name="port_name">${port_name}</param>
-            <param name="baud_rate">4000000</param>
+            <param name="baud_rate">6250000</param>
             <param name="error_timeout_ms">500</param>
             <param name="dynamixel_model_folder">/param/dxl_model</param>
-            <param name="number_of_joints">7</param>
-            <param name="number_of_transmissions">7</param>
+            <param name="number_of_joints">6</param>
+            <param name="number_of_transmissions">6</param>
             <param name="disable_torque_at_init">true</param>
             <param name="dynamixel_state_pub_msg_name">dynamixel_hardware_interface/dxl_state</param>
@@ -68,10 +68,16 @@
         <state_interface name="effort"/>
       </joint>
-      <joint name="${prefix}rh_r1_joint">
-        <command_interface name="effort"/>
-        <state_interface name="position"/>
-        <state_interface name="velocity"/>
-        <state_interface name="effort"/>
-      </joint>
+      <gpio name="omy_hat">
+        <param name="type">controller</param>
+        <param name="ID">200</param>
+        <param name="Power Enable">1</param>
+        <param name="Voltage Control Enable">1</param>
+        <param name="R LED">200</param>
+        <param name="G LED">200</param>
+        <param name="B LED">120</param>
+        <param name="Baud Rate (Bus)">8</param>
+        <param name="DXL Baud Rate">8</param>
+        <param name="Status">0</param>
+      </gpio>
       <gpio name="dxl1">
         <param name="type">dxl</param>
@@ -81,8 +87,19 @@
         <state_interface name="Present Velocity"/>
         <state_interface name="Present Current"/>
-        <param name="Drive Mode">0</param>
-        <param name="Operating Mode">0</param>
-        <param name="Return Delay Time">0</param>
-        <param name="Baud Rate">6</param>
+        <param name="Torque Enable">1</param>
+        <param name="Drive Mode">4</param>
+        <param name="Velocity Limit">3591</param>
+        <param name="Acceleration Limit">8050</param>
+        <param name="Profile Velocity">3591</param>
+        <param name="Profile Acceleration">8050</param>
+        <param name="Homing Offset">0</param>
+        <param name="Return Delay Time">0</param>
+        <param name="Position P Gain">1583185</param>
+        <param name="Velocity P Gain">41387</param>
+        <param name="Velocity I Gain">1565630</param>
+        <param name="Operating Mode">0</param>
+        <param name="Profile Acceleration Time">20</param>
+        <param name="Profile Time">40</param>
+        <param name="Bus Watchdog">1</param>
       </gpio>
       <gpio name="dxl2">
@@ -93,8 +110,18 @@
         <state_interface name="Present Velocity"/>
         <state_interface name="Present Current"/>
-        <param name="Drive Mode">1</param>
-        <param name="Operating Mode">0</param>
-        <param name="Return Delay Time">0</param>
-        <param name="Baud Rate">6</param>
+        <param name="Torque Enable">1</param>
+        <param name="Drive Mode">5</param>
+        <param name="Velocity Limit">3591</param>
+        <param name="Acceleration Limit">8050</param>
+        <param name="Profile Velocity">3591</param>
+        <param name="Profile Acceleration">8050</param>
+        <param name="Return Delay Time">0</param>
+        <param name="Position P Gain">1583185</param>
+        <param name="Velocity P Gain">41387</param>
+        <param name="Velocity I Gain">1565630</param>
+        <param name="Operating Mode">0</param>
+        <param name="Profile Acceleration Time">20</param>
+        <param name="Profile Time">40</param>
+        <param name="Bus Watchdog">1</param>
       </gpio>
       <gpio name="dxl3">
@@ -105,8 +132,18 @@
         <state_interface name="Present Velocity"/>
         <state_interface name="Present Current"/>
-        <param name="Drive Mode">0</param>
-        <param name="Operating Mode">0</param>
-        <param name="Return Delay Time">0</param>
-        <param name="Baud Rate">6</param>
+        <param name="Torque Enable">1</param>
+        <param name="Drive Mode">4</param>
+        <param name="Velocity Limit">6486</param>
+        <param name="Acceleration Limit">8050</param>
+        <param name="Profile Velocity">6486</param>
+        <param name="Profile Acceleration">8050</param>
+        <param name="Return Delay Time">0</param>
+        <param name="Position P Gain">1583185</param>
+        <param name="Velocity P Gain">18184</param>
+        <param name="Velocity I Gain">1585331</param>
+        <param name="Operating Mode">0</param>
+        <param name="Profile Acceleration Time">20</param>
+        <param name="Profile Time">40</param>
+        <param name="Bus Watchdog">1</param>
       </gpio>
       <gpio name="dxl4">
@@ -117,8 +154,18 @@
         <state_interface name="Present Velocity"/>
         <state_interface name="Present Current"/>
-        <param name="Drive Mode">1</param>
-        <param name="Operating Mode">0</param>
-        <param name="Return Delay Time">0</param>
-        <param name="Baud Rate">6</param>
+        <param name="Torque Enable">1</param>
+        <param name="Drive Mode">5</param>
+        <param name="Velocity Limit">6486</param>
+        <param name="Acceleration Limit">8050</param>
+        <param name="Profile Velocity">6486</param>
+        <param name="Profile Acceleration">8050</param>
+        <param name="Return Delay Time">0</param>
+        <param name="Position P Gain">1583185</param>
+        <param name="Velocity P Gain">18184</param>
+        <param name="Velocity I Gain">1585331</param>
+        <param name="Operating Mode">0</param>
+        <param name="Profile Acceleration Time">20</param>
+        <param name="Profile Time">40</param>
+        <param name="Bus Watchdog">1</param>
       </gpio>
       <gpio name="dxl5">
@@ -129,8 +176,18 @@
         <state_interface name="Present Velocity"/>
         <state_interface name="Present Current"/>
-        <param name="Drive Mode">0</param>
-        <param name="Operating Mode">0</param>
-        <param name="Return Delay Time">0</param>
-        <param name="Baud Rate">6</param>
+        <param name="Torque Enable">1</param>
+        <param name="Drive Mode">4</param>
+        <param name="Velocity Limit">6486</param>
+        <param name="Acceleration Limit">8050</param>
+        <param name="Profile Velocity">6486</param>
+        <param name="Profile Acceleration">8050</param>
+        <param name="Return Delay Time">0</param>
+        <param name="Position P Gain">1583185</param>
+        <param name="Velocity P Gain">18184</param>
+        <param name="Velocity I Gain">1585331</param>
+        <param name="Operating Mode">0</param>
+        <param name="Profile Acceleration Time">20</param>
+        <param name="Profile Time">40</param>
+        <param name="Bus Watchdog">1</param>
       </gpio>
       <gpio name="dxl6">
@@ -141,20 +198,18 @@
         <state_interface name="Present Velocity"/>
         <state_interface name="Present Current"/>
-        <param name="Drive Mode">1</param>
-        <param name="Operating Mode">0</param>
-        <param name="Return Delay Time">0</param>
-        <param name="Baud Rate">6</param>
-      </gpio>
-      <gpio name="dxl7">
-        <param name="type">dxl</param>
-        <param name="ID">7</param>
-        <command_interface name="Goal Current"/>
-        <state_interface name="Present Position"/>
-        <state_interface name="Present Velocity"/>
-        <state_interface name="Present Current"/>
-        <param name="Drive Mode">0</param>
-        <param name="Operating Mode">0</param>
-        <param name="Return Delay Time">0</param>
-        <param name="Baud Rate">6</param>
+        <param name="Torque Enable">1</param>
+        <param name="Drive Mode">5</param>
+        <param name="Velocity Limit">6486</param>
+        <param name="Acceleration Limit">8050</param>
+        <param name="Profile Velocity">6486</param>
+        <param name="Profile Acceleration">8050</param>
+        <param name="Return Delay Time">0</param>
+        <param name="Position P Gain">1583185</param>
+        <param name="Velocity P Gain">18184</param>
+        <param name="Velocity I Gain">1585331</param>
+        <param name="Operating Mode">0</param>
+        <param name="Profile Acceleration Time">20</param>
+        <param name="Profile Time">40</param>
+        <param name="Bus Watchdog">1</param>
       </gpio>
     </ros2_control>

File: open_manipulator_description/urdf/omy_f3m/omy_f3m.urdf.xacro (robot description, xacro)
@@ -6,5 +6,5 @@
   <xacro:arg name="mock_sensor_commands" default="false" />
   <xacro:arg name="config_type" default="omy_f3m" />
-  <xacro:arg name="ros2_control_type" default="omy_f3m_position" />
+  <xacro:arg name="ros2_control_type" default="omy_f3m_current" />
   <xacro:include filename="$(find open_manipulator_description)/urdf/omy_f3m/omy_f3m_arm.urdf.xacro" />
   <xacro:include filename="$(find open_manipulator_description)/gazebo/omy_f3m.gazebo.xacro" />
@@ -53,8 +53,17 @@
     use_mock_hardware="$(arg use_mock_hardware)"
     mock_sensor_commands="$(arg mock_sensor_commands)"/>
-  <gazebo>
-    <plugin filename="gz_ros2_control-system" name="gz_ros2_control::GazeboSimROS2ControlPlugin">
-      <parameters>$(find open_manipulator_bringup)/config/$(arg config_type)/hardware_controller_manager.yaml</parameters>
-    </plugin>
+  <xacro:if value="$(arg use_sim)">
+    <gazebo>
+      <plugin filename="gz_ros2_control-system" name="gz_ros2_control::GazeboSimROS2ControlPlugin">
+        <parameters>$(find open_manipulator_bringup)/config/$(arg config_type)/hardware_controller_manager.yaml</parameters>
+        <update_rate>400.0</update_rate>
+      </plugin>
+    </gazebo>
+  </xacro:if>
+  <!-- <gazebo reference="$(arg prefix)link3">
+    <self_collision>true</self_collision>
   </gazebo>
+  <gazebo reference="$(arg prefix)link4">
+    <self_collision>true</self_collision>
+  </gazebo> -->
 </robot>
